File: kicad/Mac DB15 to VGA TH v1.1.kicad_pcb (KiCad board)
At the start: 2 copper layers, 44.5 x 39.6 mm, 12 parts, among them J1 Mac_DB15_Male_MountingHoles, J2 VGA_DB15_Female_HighDensity_M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

Commit message: Update all projects to Kicad 6.Remove unused snapeda footprint and symbol library references.
Other:
- net class Default removed
